File: marklin 8-port bus connector.sch (EAGLE design)
At the start: 10 parts, among them J1 34V 5A, J10 34V 5A, J2 34V 5A, J3 34V 5A, J4 34V 5A, J5 34V 5A, J6 34V 5A, J7 34V 5A, J8 34V 5A, J9 34V 5A

Commit message: Update connectors
Parts:
- J1, J10, J2, J3, J4, J5, J6, J7, J8, J9: MF (none) -> WURTH ELEKTRONIK; MPN (none) -> 691111710002; OC_NEWARK (none) -> 19P1416
